File: read_a.kicad_sch (KiCad schematic)
At the start: 284 parts, among them J1 Bus_PCI_Express_x16, J10 Conn_01x05, J4 Conn_02x32_Odd_Even, J5 Conn_02x32_Odd_Even, J6 Conn_02x05_Odd_Even, J7 Conn_02x05_Odd_Even, J8 Conn_02x05_Odd_Even, J9 Conn_02x05_Odd_Even

Commit message: Schematic mostly finished.  Still need to make the PCIe connector layouts.
Parts:
- added J29: Bus_PCI_Express_x16, Connector_PCBEdge:BUS_PCIexpress_x16, symbol Connector:Bus_PCI_Express_x16
Connections:
- net +12V: now also J29.A2 (+12V), J29.A3 (+12V), J29.B1 (+12V), J29.B2 (+12V), J29.B3 (+12V)
- net +3V3: now also J29.A10 (+3.3V), J29.A9 (+3.3V), J29.B10 (3.3Vaux), J29.B8 (+3.3V)
- net CLK_PH0: now also J29.A13 (REFCLK+)
- net CLK_PH1: now also J29.A14 (REFCLK-)
- net GND: now also J29.A12 (GND), J29.A15 (GND), J29.A18 (GND), J29.A20 (GND), J29.A23 (GND), J29.A24 (GND), J29.A27 (GND), J29.A28 (GND), J29.A31 (GND), J29.A34 (GND), J29.A37 (GND), J29.A38 (GND), J29.A4 (GND), J29.A41 (GND), J29.A42 (GND), J29.A45 (GND), J29.A46 (GND), J29.A49 (GND), J29.A51 (GND), J29.A54 (GND), J29.A55 (GND), J29.A58 (GND), J29.A59 (GND), J29.A62 (GND), J29.A63 (GND), J29.A66 (GND), J29.A67 (GND), J29.A70 (GND), J29.A71 (GND), J29.A74 (GND), J29.A75 (GND), J29.A78 (GND), J29.A79 (GND), J29.A82 (GND), J29.B13 (GND), J29.B16 (GND), J29.B18 (GND), J29.B21 (GND), J29.B22 (GND), J29.B25 (GND), J29.B26 (GND), J29.B29 (GND), J29.B32 (GND), J29.B35 (GND), J29.B36 (GND), J29.B39 (GND), J29.B4 (GND), J29.B40 (GND), J29.B43 (GND), J29.B44 (GND), J29.B47 (GND), J29.B49 (GND), J29.B52 (GND), J29.B53 (GND), J29.B56 (GND), J29.B57 (GND), J29.B60 (GND), J29.B61 (GND), J29.B64 (GND), J29.B65 (GND), J29.B68 (GND), J29.B69 (GND), J29.B7 (GND), J29.B72 (GND), J29.B73 (GND), J29.B76 (GND), J29.B77 (GND), J29.B80 (GND)
- net reada0: now also J29.B14 (PETp0)
- net reada1: now also J29.B15 (PETn0)
- net reada10: now also J29.B37 (PETp5)
- net reada11: now also J29.B38 (PETn5)
- net reada12: now also J29.B41 (PETp6)
- net reada13: now also J29.B42 (PETn6)
- net reada14: now also J29.B45 (PETp7)
- net reada15: now also J29.B46 (PETn7)
- net reada16: now also D33.1 (K), D34.2 (A), J29.B50 (PETp8)
- net reada17: now also D35.1 (K), D36.2 (A), J29.B51 (PETn8)
- net reada18: now also D37.1 (K), D38.2 (A), J29.B54 (PETp9)
- net reada19: now also D39.1 (K), D40.2 (A), J29.B55 (PETn9)
- net reada2: now also J29.B19 (PETp1)
- net reada20: now also D41.1 (K), D42.2 (A), J29.B58 (PETp10)
- net reada21: now also D43.1 (K), D44.2 (A), J29.B59 (PETn10)
- net reada22: now also D45.1 (K), D46.2 (A), J29.B62 (PETp11)
- net reada23: now also D47.1 (K), D48.2 (A), J29.B63 (PETn11)
- net reada24: now also D49.1 (K), D50.2 (A), J29.B66 (PETp12)
- net reada25: now also D51.1 (K), D52.2 (A), J29.B67 (PETn12)
- net reada26: now also D53.1 (K), D54.2 (A), J29.B70 (PETp13)
- net reada27: now also D55.1 (K), D56.2 (A), J29.B71 (PETn13)
- net reada28: now also D57.1 (K), D58.2 (A), J29.B74 (PETp14)
- net reada29: now also D59.1 (K), D60.2 (A), J29.B75 (PETn14)
- net reada3: now also J29.B20 (PETn1)
- net reada30: now also D61.1 (K), D62.2 (A), J29.B78 (PETp15)
- net reada31: now also D63.1 (K), D64.2 (A), J29.B79 (PETn15)
- net reada32: now also D65.1 (K), D66.2 (A), J29.A16 (PERp0)
- net reada33: now also D67.1 (K), D68.2 (A), J29.A17 (PERn0)
- net reada34: now also D69.1 (K), D70.2 (A), J29.A21 (PERp1)
- net reada35: now also D71.1 (K), D72.2 (A), J29.A22 (PERn1)
- net reada36: now also D73.1 (K), D74.2 (A), J29.A25 (PERp2)
- net reada37: now also D75.1 (K), D76.2 (A), J29.A26 (PERn2)
- net reada38: now also D77.1 (K), D78.2 (A), J29.A29 (PERp3)
- net reada39: now also D79.1 (K), D80.2 (A), J29.A30 (PERn3)
- net reada4: now also J29.B23 (PETp2)
- net reada40: now also D81.1 (K), D82.2 (A), J29.A35 (PERp4)
- net reada41: now also D83.1 (K), D84.2 (A), J29.A36 (PERn4)
- net reada42: now also D85.1 (K), D86.2 (A), J29.A39 (PERp5)
- net reada43: now also D87.1 (K), D88.2 (A), J29.A40 (PERn5)
- net reada44: now also D89.1 (K), D90.2 (A), J29.A43 (PERp6)
- net reada45: now also D91.1 (K), D92.2 (A), J29.A44 (PERn6)
- net reada46: now also D93.1 (K), D94.2 (A), J29.A47 (PERp7)
- net reada47: now also D95.1 (K), D96.2 (A), J29.A48 (PERn7)
- net reada48: now also D97.1 (K), D98.2 (A), J29.A52 (PERp8)
- net reada49: now also D100.2 (A), D99.1 (K), J29.A53 (PERn8)
- net reada5: now also J29.B24 (PETn2)
- net reada50: now also D101.1 (K), D102.2 (A), J29.A56 (PERp9)
- net reada51: now also D103.1 (K), D104.2 (A), J29.A57 (PERn9)
- net reada52: now also D105.1 (K), D106.2 (A), J29.A60 (PERp10)
- net reada53: now also D107.1 (K), D108.2 (A), J29.A61 (PERn10)
- net reada54: now also D109.1 (K), D110.2 (A), J29.A64 (PERp11)
- net reada55: now also D111.1 (K), D112.2 (A), J29.A65 (PERn11)
- net reada56: now also D113.1 (K), D114.2 (A), J29.A68 (PERp12)
- net reada57: now also D115.1 (K), D116.2 (A), J29.A69 (PERn12)
- net reada58: now also D117.1 (K), D118.2 (A), J29.A72 (PERp13)
- net reada59: now also D119.1 (K), D120.2 (A), J29.A73 (PERn13)
- net reada6: now also J29.B27 (PETp3)
- net reada60: now also D121.1 (K), D122.2 (A), J29.A76 (PERp14)
- net reada61: now also D123.1 (K), D124.2 (A), J29.A77 (PERn14)
- net reada62: now also D125.1 (K), D126.2 (A), J29.A80 (PERp15)
- net reada63: now also D127.1 (K), D128.2 (A), J29.A81 (PERn15)
- net reada7: now also J29.B28 (PETn3)
- net reada8: now also J29.B33 (PETp4)
- net reada9: now also J29.B34 (PETn4)
- net readasel0: now also D129.1 (K), D130.2 (A), J29.B9 (JTAG1)
- net readasel1: now also D131.1 (K), D132.2 (A), J29.A5 (JTAG2)
- net readasel2: now also D133.1 (K), D134.2 (A), J29.A6 (JTAG3)
- net readasel3: now also D135.1 (K), D136.2 (A), J29.A7 (JTAG4)
- net readasel4: now also D137.1 (K), D138.2 (A), J29.A8 (JTAG5)
- net rsvda0: now also J29.B82 (RSVD)
- net rsvda1: now also J29.A50 (RSVD)
- net rsvda2: now also J29.A33 (RSVD)
- net rsvda3: now also J29.B30 (RSVD)
- net rsvda4: now also J29.A32 (RSVD)
- net rsvda5: now also J29.A19 (RSVD)
- net rsvda6: now also J29.B12 (RSVD)
- net smclka: now also J29.B5 (SMCLK)
- net smdata: now also J29.B6 (SMDAT)
- net ~{RDT}: now also J29.A11 (~{PERST})
- net ~{wakea}: now also J29.B11 (~{WAKE})
- net ~{prsnt1}: now reaches J1.A1 (~{PRSNT1}), J7.1 (Pin_1)
- net ~{prsnt1}: now also J29.A1 (~{PRSNT1})
- net ~{prsnt2}: now reaches J1.B17 (~{PRSNT2}), J7.3 (Pin_3)
- net ~{prsnt2}: now also J29.B17 (~{PRSNT2})
- net ~{prsnt3}: now reaches J1.B31 (~{PRSNT2}), J7.5 (Pin_5)
- net ~{prsnt3}: now also J29.B31 (~{PRSNT2})
- net ~{prsnt4}: now reaches J1.B48 (~{PRSNT2}), J7.7 (Pin_7)
- net ~{prsnt4}: now also J29.B48 (~{PRSNT2})
- net ~{prsnt5}: now reaches J1.B81 (~{PRSNT2}), J7.9 (Pin_9)
- net ~{prsnt5}: now also J29.B81 (~{PRSNT2})
Other:
- moved on the sheet: J1, J10, J4, J5, J6, J7, J8, J9
