File: read_b.kicad_sch (KiCad schematic)
At the start: 1 part, among them J2 Bus_PCI_Express_x16

Commit message: Schematic mostly finished.  Still need to make the PCIe connector layouts.
Parts:
- removed J2: Bus_PCI_Express_x16, Connector_PCBEdge:BUS_PCIexpress_x16, symbol Connector:Bus_PCI_Express_x16
- added D139, D141, D143, D145, D147, D149, D151, D153, D155, D157, D159, D161, D163, D165, D167, D169, D171, D173, D175, D177, D179, D181, D183, D185, D187, D189, D191, D193, D195, D197, D199, D201, D203, D205, D207, D209, D211, D213, D215, D217, D219, D221, D223, D225, D227, D229, D231, D233, D235, D237, D239, D241, D243, D245, D247, D249, D251, D253, D255, D257, D259, D261, D263, D265, D267, D269, D271, D273, D275: LED AMBER, symbol Device:LED
- added D140, D142, D144, D146, D148, D150, D152, D154, D156, D158, D160, D162, D164, D166, D168, D170, D172, D174, D176, D178, D180, D182, D184, D186, D188, D190, D192, D194, D196, D198, D200, D202, D204, D206, D208, D210, D212, D214, D216, D218, D220, D222, D224, D226, D228, D230, D232, D234, D236, D238, D240, D242, D244, D246, D248, D250, D252, D254, D256, D258, D260, D262, D264, D266, D268, D270, D272, D274, D276: LED GREEN, symbol Device:LED
- added J11, J14, J15, J2: Conn_02x05_Odd_Even, symbol Connector_Generic:Conn_02x05_Odd_Even
- added J12, J16: Conn_02x32_Odd_Even, symbol Connector_Generic:Conn_02x32_Odd_Even
- added J13, J28: Bus_PCI_Express_x16, Connector_PCBEdge:BUS_PCIexpress_x16, symbol Connector:Bus_PCI_Express_x16
- added J17: Conn_01x05, symbol Connector_Generic:Conn_01x05
- added R139, R140, R141, R142, R143, R144, R145, R146, R147, R148, R149, R150, R151, R152, R153, R154, R155, R156, R157, R158, R159, R160, R161, R162, R163, R164, R165, R166, R167, R168, R169, R170, R171, R172, R173, R174, R175, R176, R177, R178, R179, R180, R181, R182, R183, R184, R185, R186, R187, R188, R189, R190, R191, R192, R193, R194, R195, R196, R197, R198, R199, R200, R201, R202, R203, R204, R205, R206, R207, R208, R209, R210, R211, R212, R213, R214, R215, R216, R217, R218, R219, R220, R221, R222, R223, R224, R225, R226, R227, R228, R229, R230, R231, R232, R233, R234, R235, R236, R237, R238, R239, R240, R241, R242, R243, R244, R245, R246, R247, R248, R249, R250, R251, R252, R253, R254, R255, R256, R257, R258, R259, R260, R261, R262, R263, R264, R265, R266, R267, R268, R269, R270, R271, R272, R273, R274, R275, R276: 1K, symbol Device:R
Connections:
- new net: D268.1 (K), R268.1
- new net: D193.2 (A), R193.2
- new net: D257.2 (A), R257.2
- new net: D253.2 (A), R253.2
- new net: D224.1 (K), R224.1
- new net: D152.1 (K), R152.1
- new net: D221.2 (A), R221.2
- new net: D187.2 (A), R187.2
- new net: D250.1 (K), R250.1
- new net: D256.1 (K), R256.1
- new net: D163.2 (A), R163.2
- new net: D178.1 (K), R178.1
- new net: D275.2 (A), R275.2
- new net: D155.2 (A), R155.2
- new net: D176.1 (K), R176.1
- new net: D265.2 (A), R265.2
- new net: D145.2 (A), R145.2
- new net: D216.1 (K), R216.1
- new net: D158.1 (K), R158.1
- new net: D214.1 (K), R214.1
- new net: D177.2 (A), R177.2
- new net: D270.1 (K), R270.1
- new net: D222.1 (K), R222.1
- new net: D207.2 (A), R207.2
- new net: D144.1 (K), R144.1
- new net: D211.2 (A), R211.2
- new net: D235.2 (A), R235.2
- new net: D269.2 (A), R269.2
- new net: D243.2 (A), R243.2
- new net: D142.1 (K), R142.1
- new net: D241.2 (A), R241.2
- new net: D218.1 (K), R218.1
- new net: D154.1 (K), R154.1
- new net: D252.1 (K), R252.1
- new net: D184.1 (K), R184.1
- new net: D274.1 (K), R274.1
- new net: D228.1 (K), R228.1
- new net: D209.2 (A), R209.2
- new net: D169.2 (A), R169.2
- new net: D183.2 (A), R183.2
- new net: D231.2 (A), R231.2
- new net: D272.1 (K), R272.1
- new net: D215.2 (A), R215.2
- new net: D198.1 (K), R198.1
- new net: D141.2 (A), R141.2
- new net: D244.1 (K), R244.1
- new net: D151.2 (A), R151.2
- new net: D202.1 (K), R202.1
- new net: D161.2 (A), R161.2
- new net: D199.2 (A), R199.2
- new net: D167.2 (A), R167.2
- new net: D262.1 (K), R262.1
- new net: D249.2 (A), R249.2
- new net: D246.1 (K), R246.1
- new net: D229.2 (A), R229.2
- new net: D191.2 (A), R191.2
- new net: D156.1 (K), R156.1
- new net: D226.1 (K), R226.1
- new net: D239.2 (A), R239.2
- new net: D251.2 (A), R251.2
- new net: D185.2 (A), R185.2
- new net: D225.2 (A), R225.2
- new net: D242.1 (K), R242.1
- new net: D157.2 (A), R157.2
- new net: D219.2 (A), R219.2
- new net: D174.1 (K), R174.1
- new net: D162.1 (K), R162.1
- new net: D273.2 (A), R273.2
- new net: D171.2 (A), R171.2
- new net: D170.1 (K), R170.1
- new net: D230.1 (K), R230.1
- new net: D166.1 (K), R166.1
- new net: D140.1 (K), R140.1
- new net: D236.1 (K), R236.1
- new net: D254.1 (K), R254.1
- new net: D165.2 (A), R165.2
- new net: D172.1 (K), R172.1
- new net: D259.2 (A), R259.2
- new net: D204.1 (K), R204.1
- new net: D180.1 (K), R180.1
- new net: D240.1 (K), R240.1
- new net: D267.2 (A), R267.2
- new net: D261.2 (A), R261.2
- new net: D238.1 (K), R238.1
- new net: D189.2 (A), R189.2
- new net: D146.1 (K), R146.1
- new net: D248.1 (K), R248.1
- new net: D220.1 (K), R220.1
- new net: D201.2 (A), R201.2
- new net: D149.2 (A), R149.2
- new net: D194.1 (K), R194.1
- new net: D212.1 (K), R212.1
- new net: D179.2 (A), R179.2
- new net: D139.2 (A), R139.2
- new net: D147.2 (A), R147.2
- new net: D264.1 (K), R264.1
- new net: D143.2 (A), R143.2
- new net: D206.1 (K), R206.1
- new net: D227.2 (A), R227.2
- new net: D237.2 (A), R237.2
- new net: D196.1 (K), R196.1
- new net: D255.2 (A), R255.2
- new net: D271.2 (A), R271.2
- new net: D195.2 (A), R195.2
- new net: D205.2 (A), R205.2
- new net: D203.2 (A), R203.2
- new net: D168.1 (K), R168.1
- new net: D148.1 (K), R148.1
- new net: D247.2 (A), R247.2
- new net: D260.1 (K), R260.1
- new net: D200.1 (K), R200.1
- new net: D190.1 (K), R190.1
- new net: D197.2 (A), R197.2
- new net: D210.1 (K), R210.1
- new net: D258.1 (K), R258.1
- new net: D160.1 (K), R160.1
- new net: D182.1 (K), R182.1
- new net: D173.2 (A), R173.2
- new net: D188.1 (K), R188.1
- new net: D150.1 (K), R150.1
- new net: D276.1 (K), R276.1
- new net: D266.1 (K), R266.1
- new net: D186.1 (K), R186.1
- new net: D233.2 (A), R233.2
- new net: D223.2 (A), R223.2
- new net: D153.2 (A), R153.2
- new net: D213.2 (A), R213.2
- new net: D181.2 (A), R181.2
- new net: D263.2 (A), R263.2
- new net: D234.1 (K), R234.1
- new net: D245.2 (A), R245.2
- new net: D159.2 (A), R159.2
- new net: D164.1 (K), R164.1
- new net: D175.2 (A), R175.2
- new net: D217.2 (A), R217.2
- new net: D232.1 (K), R232.1
- new net: D192.1 (K), R192.1
- new net: D208.1 (K), R208.1
- new net +12V: J13.A2 (+12V), J13.A3 (+12V), J13.B1 (+12V), J13.B2 (+12V), J13.B3 (+12V), J28.A2 (+12V), J28.A3 (+12V), J28.B1 (+12V), J28.B2 (+12V), J28.B3 (+12V)
- new net +3V3: J13.A10 (+3.3V), J13.A9 (+3.3V), J13.B10 (3.3Vaux), J13.B8 (+3.3V), J17.1 (Pin_1), J17.2 (Pin_2), J17.3 (Pin_3), J17.4 (Pin_4), J17.5 (Pin_5), J28.A10 (+3.3V), J28.A9 (+3.3V), J28.B10 (3.3Vaux), J28.B8 (+3.3V), R139.1, R141.1, R143.1, R145.1, R147.1, R149.1, R151.1, R153.1, R155.1, R157.1, R159.1, R161.1, R163.1, R165.1, R167.1, R169.1, R171.1, R173.1, R175.1, R177.1, R179.1, R181.1, R183.1, R185.1, R187.1, R189.1, R191.1, R193.1, R195.1, R197.1, R199.1, R201.1, R203.1, R205.1, R207.1, R209.1, R211.1, R213.1, R215.1, R217.1, R219.1, R221.1, R223.1, R225.1, R227.1, R229.1, R231.1, R233.1, R235.1, R237.1, R239.1, R241.1, R243.1, R245.1, R247.1, R249.1, R251.1, R253.1, R255.1, R257.1, R259.1, R261.1, R263.1, R265.1, R267.1, R269.1, R271.1, R273.1, R275.1
- new net CLK_PH0: J13.A13 (REFCLK+), J28.A13 (REFCLK+)
- new net CLK_PH1: J13.A14 (REFCLK-), J28.A14 (REFCLK-)
- new net GND: J11.10 (Pin_10), J11.2 (Pin_2), J11.4 (Pin_4), J11.6 (Pin_6), J11.8 (Pin_8), J12.10 (Pin_10), J12.12 (Pin_12), J12.14 (Pin_14), J12.16 (Pin_16), J12.18 (Pin_18), J12.2 (Pin_2), J12.20 (Pin_20), J12.22 (Pin_22), J12.24 (Pin_24), J12.26 (Pin_26), J12.28 (Pin_28), J12.30 (Pin_30), J12.32 (Pin_32), J12.34 (Pin_34), J12.36 (Pin_36), J12.38 (Pin_38), J12.4 (Pin_4), J12.40 (Pin_40), J12.42 (Pin_42), J12.44 (Pin_44), J12.46 (Pin_46), J12.48 (Pin_48), J12.50 (Pin_50), J12.52 (Pin_52), J12.54 (Pin_54), J12.56 (Pin_56), J12.58 (Pin_58), J12.6 (Pin_6), J12.60 (Pin_60), J12.62 (Pin_62), J12.64 (Pin_64), J12.8 (Pin_8), J13.A12 (GND), J13.A15 (GND), J13.A18 (GND), J13.A20 (GND), J13.A23 (GND), J13.A24 (GND), J13.A27 (GND), J13.A28 (GND), J13.A31 (GND), J13.A34 (GND), J13.A37 (GND), J13.A38 (GND), J13.A4 (GND), J13.A41 (GND), J13.A42 (GND), J13.A45 (GND), J13.A46 (GND), J13.A49 (GND), J13.A51 (GND), J13.A54 (GND), J13.A55 (GND), J13.A58 (GND), J13.A59 (GND), J13.A62 (GND), J13.A63 (GND), J13.A66 (GND), J13.A67 (GND), J13.A70 (GND), J13.A71 (GND), J13.A74 (GND), J13.A75 (GND), J13.A78 (GND), J13.A79 (GND), J13.A82 (GND), J13.B13 (GND), J13.B16 (GND), J13.B18 (GND), J13.B21 (GND), J13.B22 (GND), J13.B25 (GND), J13.B26 (GND), J13.B29 (GND), J13.B32 (GND), J13.B35 (GND), J13.B36 (GND), J13.B39 (GND), J13.B4 (GND), J13.B40 (GND), J13.B43 (GND), J13.B44 (GND), J13.B47 (GND), J13.B49 (GND), J13.B52 (GND), J13.B53 (GND), J13.B56 (GND), J13.B57 (GND), J13.B60 (GND), J13.B61 (GND), J13.B64 (GND), J13.B65 (GND), J13.B68 (GND), J13.B69 (GND), J13.B7 (GND), J13.B72 (GND), J13.B73 (GND), J13.B76 (GND), J13.B77 (GND), J13.B80 (GND), J14.10 (Pin_10), J14.2 (Pin_2), J14.4 (Pin_4), J14.6 (Pin_6), J14.8 (Pin_8), J15.10 (Pin_10), J15.2 (Pin_2), J15.4 (Pin_4), J15.6 (Pin_6), J15.8 (Pin_8), J16.10 (Pin_10), J16.12 (Pin_12), J16.14 (Pin_14), J16.16 (Pin_16), J16.18 (Pin_18), J16.2 (Pin_2), J16.20 (Pin_20), J16.22 (Pin_22), J16.24 (Pin_24), J16.26 (Pin_26), J16.28 (Pin_28), J16.30 (Pin_30), J16.32 (Pin_32), J16.34 (Pin_34), J16.36 (Pin_36), J16.38 (Pin_38), J16.4 (Pin_4), J16.40 (Pin_40), J16.42 (Pin_42), J16.44 (Pin_44), J16.46 (Pin_46), J16.48 (Pin_48), J16.50 (Pin_50), J16.52 (Pin_52), J16.54 (Pin_54), J16.56 (Pin_56), J16.58 (Pin_58), J16.6 (Pin_6), J16.60 (Pin_60), J16.62 (Pin_62), J16.64 (Pin_64), J16.8 (Pin_8), J2.10 (Pin_10), J2.2 (Pin_2), J2.4 (Pin_4), J2.6 (Pin_6), J2.8 (Pin_8), J28.A12 (GND), J28.A15 (GND), J28.A18 (GND), J28.A20 (GND), J28.A23 (GND), J28.A24 (GND), J28.A27 (GND), J28.A28 (GND), J28.A31 (GND), J28.A34 (GND), J28.A37 (GND), J28.A38 (GND), J28.A4 (GND), J28.A41 (GND), J28.A42 (GND), J28.A45 (GND), J28.A46 (GND), J28.A49 (GND), J28.A51 (GND), J28.A54 (GND), J28.A55 (GND), J28.A58 (GND), J28.A59 (GND), J28.A62 (GND), J28.A63 (GND), J28.A66 (GND), J28.A67 (GND), J28.A70 (GND), J28.A71 (GND), J28.A74 (GND), J28.A75 (GND), J28.A78 (GND), J28.A79 (GND), J28.A82 (GND), J28.B13 (GND), J28.B16 (GND), J28.B18 (GND), J28.B21 (GND), J28.B22 (GND), J28.B25 (GND), J28.B26 (GND), J28.B29 (GND), J28.B32 (GND), J28.B35 (GND), J28.B36 (GND), J28.B39 (GND), J28.B4 (GND), J28.B40 (GND), J28.B43 (GND), J28.B44 (GND), J28.B47 (GND), J28.B49 (GND), J28.B52 (GND), J28.B53 (GND), J28.B56 (GND), J28.B57 (GND), J28.B60 (GND), J28.B61 (GND), J28.B64 (GND), J28.B65 (GND), J28.B68 (GND), J28.B69 (GND), J28.B7 (GND), J28.B72 (GND), J28.B73 (GND), J28.B76 (GND), J28.B77 (GND), J28.B80 (GND), R140.2, R142.2, R144.2, R146.2, R148.2, R150.2, R152.2, R154.2, R156.2, R158.2, R160.2, R162.2, R164.2, R166.2, R168.2, R170.2, R172.2, R174.2, R176.2, R178.2, R180.2, R182.2, R184.2, R186.2, R188.2, R190.2, R192.2, R194.2, R196.2, R198.2, R200.2, R202.2, R204.2, R206.2, R208.2, R210.2, R212.2, R214.2, R216.2, R218.2, R220.2, R222.2, R224.2, R226.2, R228.2, R230.2, R232.2, R234.2, R236.2, R238.2, R240.2, R242.2, R244.2, R246.2, R248.2, R250.2, R252.2, R254.2, R256.2, R258.2, R260.2, R262.2, R264.2, R266.2, R268.2, R270.2, R272.2, R274.2, R276.2
- new net readb0: D149.1 (K), D150.2 (A), J12.1 (Pin_1), J13.B14 (PETp0), J28.B14 (PETp0)
- new net readb1: D157.1 (K), D158.2 (A), J12.3 (Pin_3), J13.B15 (PETn0), J28.B15 (PETn0)
- new net readb10: D229.1 (K), D230.2 (A), J12.21 (Pin_21), J13.B37 (PETp5), J28.B37 (PETp5)
- new net readb11: D237.1 (K), D238.2 (A), J12.23 (Pin_23), J13.B38 (PETn5), J28.B38 (PETn5)
- new net readb12: D245.1 (K), D246.2 (A), J12.25 (Pin_25), J13.B41 (PETp6), J28.B41 (PETp6)
- new net readb13: D253.1 (K), D254.2 (A), J12.27 (Pin_27), J13.B42 (PETn6), J28.B42 (PETn6)
- new net readb14: D261.1 (K), D262.2 (A), J12.29 (Pin_29), J13.B45 (PETp7), J28.B45 (PETp7)
- new net readb15: D269.1 (K), D270.2 (A), J12.31 (Pin_31), J13.B46 (PETn7), J28.B46 (PETn7)
- new net readb16: D151.1 (K), D152.2 (A), J12.33 (Pin_33), J13.B50 (PETp8), J28.B50 (PETp8)
- new net readb17: D159.1 (K), D160.2 (A), J12.35 (Pin_35), J13.B51 (PETn8), J28.B51 (PETn8)
- new net readb18: D167.1 (K), D168.2 (A), J12.37 (Pin_37), J13.B54 (PETp9), J28.B54 (PETp9)
- new net readb19: D175.1 (K), D176.2 (A), J12.39 (Pin_39), J13.B55 (PETn9), J28.B55 (PETn9)
- new net readb2: D165.1 (K), D166.2 (A), J12.5 (Pin_5), J13.B19 (PETp1), J28.B19 (PETp1)
- new net readb20: D183.1 (K), D184.2 (A), J12.41 (Pin_41), J13.B58 (PETp10), J28.B58 (PETp10)
- new net readb21: D191.1 (K), D192.2 (A), J12.43 (Pin_43), J13.B59 (PETn10), J28.B59 (PETn10)
- new net readb22: D199.1 (K), D200.2 (A), J12.45 (Pin_45), J13.B62 (PETp11), J28.B62 (PETp11)
- new net readb23: D207.1 (K), D208.2 (A), J12.47 (Pin_47), J13.B63 (PETn11), J28.B63 (PETn11)
- new net readb24: D215.1 (K), D216.2 (A), J12.49 (Pin_49), J13.B66 (PETp12), J28.B66 (PETp12)
- new net readb25: D223.1 (K), D224.2 (A), J12.51 (Pin_51), J13.B67 (PETn12), J28.B67 (PETn12)
- new net readb26: D231.1 (K), D232.2 (A), J12.53 (Pin_53), J13.B70 (PETp13), J28.B70 (PETp13)
- new net readb27: D239.1 (K), D240.2 (A), J12.55 (Pin_55), J13.B71 (PETn13), J28.B71 (PETn13)
- new net readb28: D247.1 (K), D248.2 (A), J12.57 (Pin_57), J13.B74 (PETp14), J28.B74 (PETp14)
- new net readb29: D255.1 (K), D256.2 (A), J12.59 (Pin_59), J13.B75 (PETn14), J28.B75 (PETn14)
- new net readb3: D173.1 (K), D174.2 (A), J12.7 (Pin_7), J13.B20 (PETn1), J28.B20 (PETn1)
- new net readb30: D263.1 (K), D264.2 (A), J12.61 (Pin_61), J13.B78 (PETp15), J28.B78 (PETp15)
- new net readb31: D271.1 (K), D272.2 (A), J12.63 (Pin_63), J13.B79 (PETn15), J28.B79 (PETn15)
- new net readb32: D153.1 (K), D154.2 (A), J13.A16 (PERp0), J16.1 (Pin_1), J28.A16 (PERp0)
- new net readb33: D161.1 (K), D162.2 (A), J13.A17 (PERn0), J16.3 (Pin_3), J28.A17 (PERn0)
- new net readb34: D169.1 (K), D170.2 (A), J13.A21 (PERp1), J16.5 (Pin_5), J28.A21 (PERp1)
- new net readb35: D177.1 (K), D178.2 (A), J13.A22 (PERn1), J16.7 (Pin_7), J28.A22 (PERn1)
- new net readb36: D185.1 (K), D186.2 (A), J13.A25 (PERp2), J16.9 (Pin_9), J28.A25 (PERp2)
- new net readb37: D193.1 (K), D194.2 (A), J13.A26 (PERn2), J16.11 (Pin_11), J28.A26 (PERn2)
- new net readb38: D201.1 (K), D202.2 (A), J13.A29 (PERp3), J16.13 (Pin_13), J28.A29 (PERp3)
- new net readb39: D209.1 (K), D210.2 (A), J13.A30 (PERn3), J16.15 (Pin_15), J28.A30 (PERn3)
- new net readb4: D181.1 (K), D182.2 (A), J12.9 (Pin_9), J13.B23 (PETp2), J28.B23 (PETp2)
- new net readb40: D217.1 (K), D218.2 (A), J13.A35 (PERp4), J16.17 (Pin_17), J28.A35 (PERp4)
- new net readb41: D225.1 (K), D226.2 (A), J13.A36 (PERn4), J16.19 (Pin_19), J28.A36 (PERn4)
- new net readb42: D233.1 (K), D234.2 (A), J13.A39 (PERp5), J16.21 (Pin_21), J28.A39 (PERp5)
- new net readb43: D241.1 (K), D242.2 (A), J13.A40 (PERn5), J16.23 (Pin_23), J28.A40 (PERn5)
- new net readb44: D249.1 (K), D250.2 (A), J13.A43 (PERp6), J16.25 (Pin_25), J28.A43 (PERp6)
- new net readb45: D257.1 (K), D258.2 (A), J13.A44 (PERn6), J16.27 (Pin_27), J28.A44 (PERn6)
- new net readb46: D265.1 (K), D266.2 (A), J13.A47 (PERp7), J16.29 (Pin_29), J28.A47 (PERp7)
- new net readb47: D273.1 (K), D274.2 (A), J13.A48 (PERn7), J16.31 (Pin_31), J28.A48 (PERn7)
- new net readb48: D155.1 (K), D156.2 (A), J13.A52 (PERp8), J16.33 (Pin_33), J28.A52 (PERp8)
- new net readb49: D163.1 (K), D164.2 (A), J13.A53 (PERn8), J16.35 (Pin_35), J28.A53 (PERn8)
- new net readb5: D189.1 (K), D190.2 (A), J12.11 (Pin_11), J13.B24 (PETn2), J28.B24 (PETn2)
- new net readb50: D171.1 (K), D172.2 (A), J13.A56 (PERp9), J16.37 (Pin_37), J28.A56 (PERp9)
- new net readb51: D179.1 (K), D180.2 (A), J13.A57 (PERn9), J16.39 (Pin_39), J28.A57 (PERn9)
- new net readb52: D187.1 (K), D188.2 (A), J13.A60 (PERp10), J16.41 (Pin_41), J28.A60 (PERp10)
- new net readb53: D195.1 (K), D196.2 (A), J13.A61 (PERn10), J16.43 (Pin_43), J28.A61 (PERn10)
- new net readb54: D203.1 (K), D204.2 (A), J13.A64 (PERp11), J16.45 (Pin_45), J28.A64 (PERp11)
- new net readb55: D211.1 (K), D212.2 (A), J13.A65 (PERn11), J16.47 (Pin_47), J28.A65 (PERn11)
- new net readb56: D219.1 (K), D220.2 (A), J13.A68 (PERp12), J16.49 (Pin_49), J28.A68 (PERp12)
- new net readb57: D227.1 (K), D228.2 (A), J13.A69 (PERn12), J16.51 (Pin_51), J28.A69 (PERn12)
- new net readb58: D235.1 (K), D236.2 (A), J13.A72 (PERp13), J16.53 (Pin_53), J28.A72 (PERp13)
- new net readb59: D243.1 (K), D244.2 (A), J13.A73 (PERn13), J16.55 (Pin_55), J28.A73 (PERn13)
- new net readb6: D197.1 (K), D198.2 (A), J12.13 (Pin_13), J13.B27 (PETp3), J28.B27 (PETp3)
- new net readb60: D251.1 (K), D252.2 (A), J13.A76 (PERp14), J16.57 (Pin_57), J28.A76 (PERp14)
- new net readb61: D259.1 (K), D260.2 (A), J13.A77 (PERn14), J16.59 (Pin_59), J28.A77 (PERn14)
- new net readb62: D267.1 (K), D268.2 (A), J13.A80 (PERp15), J16.61 (Pin_61), J28.A80 (PERp15)
- new net readb63: D275.1 (K), D276.2 (A), J13.A81 (PERn15), J16.63 (Pin_63), J28.A81 (PERn15)
- new net readb7: D205.1 (K), D206.2 (A), J12.15 (Pin_15), J13.B28 (PETn3), J28.B28 (PETn3)
- new net readb8: D213.1 (K), D214.2 (A), J12.17 (Pin_17), J13.B33 (PETp4), J28.B33 (PETp4)
- new net readb9: D221.1 (K), D222.2 (A), J12.19 (Pin_19), J13.B34 (PETn4), J28.B34 (PETn4)
- new net readbsel0: D139.1 (K), D140.2 (A), J13.B9 (JTAG1), J15.1 (Pin_1), J28.B9 (JTAG1)
- new net readbsel1: D141.1 (K), D142.2 (A), J13.A5 (JTAG2), J15.3 (Pin_3), J28.A5 (JTAG2)
- new net readbsel2: D143.1 (K), D144.2 (A), J13.A6 (JTAG3), J15.5 (Pin_5), J28.A6 (JTAG3)
- new net readbsel3: D145.1 (K), D146.2 (A), J13.A7 (JTAG4), J15.7 (Pin_7), J28.A7 (JTAG4)
- new net readbsel4: D147.1 (K), D148.2 (A), J13.A8 (JTAG5), J15.9 (Pin_9), J28.A8 (JTAG5)
- new net rsvda0: J13.B82 (RSVD), J14.1 (Pin_1), J28.B82 (RSVD)
- new net rsvda1: J13.A50 (RSVD), J14.3 (Pin_3), J28.A50 (RSVD)
- new net rsvda2: J13.A33 (RSVD), J14.5 (Pin_5), J28.A33 (RSVD)
- new net rsvda3: J13.B30 (RSVD), J14.7 (Pin_7), J28.B30 (RSVD)
- new net rsvda4: J13.A32 (RSVD), J14.9 (Pin_9), J28.A32 (RSVD)
- new net rsvda5: J13.A19 (RSVD), J2.1 (Pin_1), J28.A19 (RSVD)
- new net rsvda6: J13.B12 (RSVD), J2.3 (Pin_3), J28.B12 (RSVD)
- new net smclka: J13.B5 (SMCLK), J2.7 (Pin_7), J28.B5 (SMCLK)
- new net smdata: J13.B6 (SMDAT), J2.9 (Pin_9), J28.B6 (SMDAT)
- new net ~{RDT}: J13.A11 (~{PERST}), J28.A11 (~{PERST})
- new net ~{prsnt1}: J11.1 (Pin_1), J13.A1 (~{PRSNT1}), J28.A1 (~{PRSNT1})
- new net ~{prsnt2}: J11.3 (Pin_3), J13.B17 (~{PRSNT2}), J28.B17 (~{PRSNT2})
- new net ~{prsnt3}: J11.5 (Pin_5), J13.B31 (~{PRSNT2}), J28.B31 (~{PRSNT2})
- new net ~{prsnt4}: J11.7 (Pin_7), J13.B48 (~{PRSNT2}), J28.B48 (~{PRSNT2})
- new net ~{prsnt5}: J11.9 (Pin_9), J13.B81 (~{PRSNT2}), J28.B81 (~{PRSNT2})
- new net ~{wakea}: J13.B11 (~{WAKE}), J2.5 (Pin_5), J28.B11 (~{WAKE})
Other:
- note added: "HI IND"
- note added: "LO IND"
