File: write.kicad_sch (KiCad schematic)
At the start: 1 part, among them J3 Bus_PCI_Express_x16

Commit message: Schematic mostly finished.  Still need to make the PCIe connector layouts.
Parts:
- removed J3: Bus_PCI_Express_x16, Connector_PCBEdge:BUS_PCIexpress_x16, symbol Connector:Bus_PCI_Express_x16
- added D277, D279, D281, D283, D285, D287, D289, D291, D293, D295, D297, D299, D301, D303, D305, D307, D309, D311, D313, D315, D317, D319, D321, D323, D325, D327, D329, D331, D333, D335, D337, D339, D341, D343, D345, D347, D349, D351, D353, D355, D357, D359, D361, D363, D365, D367, D369, D371, D373, D375, D377, D379, D381, D383, D385, D387, D389, D391, D393, D395, D397, D399, D401, D403, D405, D407, D409, D411, D413: LED AMBER, symbol Device:LED
- added D278, D280, D282, D284, D286, D288, D290, D292, D294, D296, D298, D300, D302, D304, D306, D308, D310, D312, D314, D316, D318, D320, D322, D324, D326, D328, D330, D332, D334, D336, D338, D340, D342, D344, D346, D348, D350, D352, D354, D356, D358, D360, D362, D364, D366, D368, D370, D372, D374, D376, D378, D380, D382, D384, D386, D388, D390, D392, D394, D396, D398, D400, D402, D404, D406, D408, D410, D412, D414: LED GREEN, symbol Device:LED
- added J18, J21, J22, J3: Conn_02x05_Odd_Even, symbol Connector_Generic:Conn_02x05_Odd_Even
- added J19, J23: Conn_02x32_Odd_Even, symbol Connector_Generic:Conn_02x32_Odd_Even
- added J20, J27: Bus_PCI_Express_x16, Connector_PCBEdge:BUS_PCIexpress_x16, symbol Connector:Bus_PCI_Express_x16
- added J24: Conn_01x05, symbol Connector_Generic:Conn_01x05
- added J25, J26: Conn_01x32, symbol Connector_Generic:Conn_01x32
- added R277, R278, R279, R280, R281, R282, R283, R284, R285, R286, R287, R288, R289, R290, R291, R292, R293, R294, R295, R296, R297, R298, R299, R300, R301, R302, R303, R304, R305, R306, R307, R308, R309, R310, R311, R312, R313, R314, R315, R316, R317, R318, R319, R320, R321, R322, R323, R324, R325, R326, R327, R328, R329, R330, R331, R332, R333, R334, R335, R336, R337, R338, R339, R340, R341, R342, R343, R344, R345, R346, R347, R348, R349, R350, R351, R352, R353, R354, R355, R356, R357, R358, R359, R360, R361, R362, R363, R364, R365, R366, R367, R368, R369, R370, R371, R372, R373, R374, R375, R376, R377, R378, R379, R380, R381, R382, R383, R384, R385, R386, R387, R388, R389, R390, R391, R392, R393, R394, R395, R396, R397, R398, R399, R400, R401, R402, R403, R404, R405, R406, R407, R408, R409, R410, R411, R412, R413, R414: 1K, symbol Device:R
Connections:
- new net: D293.2 (A), R293.2
- new net: D370.1 (K), R370.1
- new net: D309.2 (A), R309.2
- new net: D304.1 (K), R304.1
- new net: D392.1 (K), R392.1
- new net: D354.1 (K), R354.1
- new net: D317.2 (A), R317.2
- new net: D391.2 (A), R391.2
- new net: D371.2 (A), R371.2
- new net: D302.1 (K), R302.1
- new net: D346.1 (K), R346.1
- new net: D285.2 (A), R285.2
- new net: D361.2 (A), R361.2
- new net: D277.2 (A), R277.2
- new net: D330.1 (K), R330.1
- new net: D288.1 (K), R288.1
- new net: D372.1 (K), R372.1
- new net: D336.1 (K), R336.1
- new net: D328.1 (K), R328.1
- new net: D319.2 (A), R319.2
- new net: D297.2 (A), R297.2
- new net: D407.2 (A), R407.2
- new net: D338.1 (K), R338.1
- new net: D347.2 (A), R347.2
- new net: D393.2 (A), R393.2
- new net: D401.2 (A), R401.2
- new net: D287.2 (A), R287.2
- new net: D305.2 (A), R305.2
- new net: D388.1 (K), R388.1
- new net: D412.1 (K), R412.1
- new net: D360.1 (K), R360.1
- new net: D295.2 (A), R295.2
- new net: D377.2 (A), R377.2
- new net: D314.1 (K), R314.1
- new net: D343.2 (A), R343.2
- new net: D278.1 (K), R278.1
- new net: D311.2 (A), R311.2
- new net: D364.1 (K), R364.1
- new net: D333.2 (A), R333.2
- new net: D402.1 (K), R402.1
- new net: D366.1 (K), R366.1
- new net: D327.2 (A), R327.2
- new net: D397.2 (A), R397.2
- new net: D307.2 (A), R307.2
- new net: D281.2 (A), R281.2
- new net: D280.1 (K), R280.1
- new net: D325.2 (A), R325.2
- new net: D414.1 (K), R414.1
- new net: D373.2 (A), R373.2
- new net: D321.2 (A), R321.2
- new net: D301.2 (A), R301.2
- new net: D351.2 (A), R351.2
- new net: D352.1 (K), R352.1
- new net: D379.2 (A), R379.2
- new net: D300.1 (K), R300.1
- new net: D406.1 (K), R406.1
- new net: D375.2 (A), R375.2
- new net: D404.1 (K), R404.1
- new net: D389.2 (A), R389.2
- new net: D359.2 (A), R359.2
- new net: D385.2 (A), R385.2
- new net: D398.1 (K), R398.1
- new net: D286.1 (K), R286.1
- new net: D410.1 (K), R410.1
- new net: D383.2 (A), R383.2
- new net: D344.1 (K), R344.1
- new net: D369.2 (A), R369.2
- new net: D323.2 (A), R323.2
- new net: D335.2 (A), R335.2
- new net: D292.1 (K), R292.1
- new net: D394.1 (K), R394.1
- new net: D279.2 (A), R279.2
- new net: D341.2 (A), R341.2
- new net: D298.1 (K), R298.1
- new net: D299.2 (A), R299.2
- new net: D384.1 (K), R384.1
- new net: D315.2 (A), R315.2
- new net: D376.1 (K), R376.1
- new net: D320.1 (K), R320.1
- new net: D390.1 (K), R390.1
- new net: D306.1 (K), R306.1
- new net: D340.1 (K), R340.1
- new net: D355.2 (A), R355.2
- new net: D349.2 (A), R349.2
- new net: D357.2 (A), R357.2
- new net: D363.2 (A), R363.2
- new net: D316.1 (K), R316.1
- new net: D296.1 (K), R296.1
- new net: D313.2 (A), R313.2
- new net: D339.2 (A), R339.2
- new net: D400.1 (K), R400.1
- new net: D283.2 (A), R283.2
- new net: D326.1 (K), R326.1
- new net: D282.1 (K), R282.1
- new net: D386.1 (K), R386.1
- new net: D353.2 (A), R353.2
- new net: D396.1 (K), R396.1
- new net: D303.2 (A), R303.2
- new net: D345.2 (A), R345.2
- new net: D362.1 (K), R362.1
- new net: D378.1 (K), R378.1
- new net: D382.1 (K), R382.1
- new net: D408.1 (K), R408.1
- new net: D342.1 (K), R342.1
- new net: D310.1 (K), R310.1
- new net: D291.2 (A), R291.2
- new net: D381.2 (A), R381.2
- new net: D403.2 (A), R403.2
- new net: D290.1 (K), R290.1
- new net: D308.1 (K), R308.1
- new net: D405.2 (A), R405.2
- new net: D409.2 (A), R409.2
- new net: D337.2 (A), R337.2
- new net: D356.1 (K), R356.1
- new net: D334.1 (K), R334.1
- new net: D380.1 (K), R380.1
- new net: D358.1 (K), R358.1
- new net: D413.2 (A), R413.2
- new net: D324.1 (K), R324.1
- new net: D365.2 (A), R365.2
- new net: D318.1 (K), R318.1
- new net: D331.2 (A), R331.2
- new net: D329.2 (A), R329.2
- new net: D294.1 (K), R294.1
- new net: D411.2 (A), R411.2
- new net: D322.1 (K), R322.1
- new net: D332.1 (K), R332.1
- new net: D312.1 (K), R312.1
- new net: D284.1 (K), R284.1
- new net: D367.2 (A), R367.2
- new net: D289.2 (A), R289.2
- new net: D348.1 (K), R348.1
- new net: D374.1 (K), R374.1
- new net: D399.2 (A), R399.2
- new net: D387.2 (A), R387.2
- new net: D350.1 (K), R350.1
- new net: D395.2 (A), R395.2
- new net: D368.1 (K), R368.1
- new net +12V: J20.A2 (+12V), J20.A3 (+12V), J20.B1 (+12V), J20.B2 (+12V), J20.B3 (+12V), J27.A2 (+12V), J27.A3 (+12V), J27.B1 (+12V), J27.B2 (+12V), J27.B3 (+12V)
- new net +3V3: J20.A10 (+3.3V), J20.A9 (+3.3V), J20.B10 (3.3Vaux), J20.B8 (+3.3V), J24.1 (Pin_1), J24.2 (Pin_2), J24.3 (Pin_3), J24.4 (Pin_4), J24.5 (Pin_5), J25.1 (Pin_1), J25.10 (Pin_10), J25.11 (Pin_11), J25.12 (Pin_12), J25.13 (Pin_13), J25.14 (Pin_14), J25.15 (Pin_15), J25.16 (Pin_16), J25.17 (Pin_17), J25.18 (Pin_18), J25.19 (Pin_19), J25.2 (Pin_2), J25.20 (Pin_20), J25.21 (Pin_21), J25.22 (Pin_22), J25.23 (Pin_23), J25.24 (Pin_24), J25.25 (Pin_25), J25.26 (Pin_26), J25.27 (Pin_27), J25.28 (Pin_28), J25.29 (Pin_29), J25.3 (Pin_3), J25.30 (Pin_30), J25.31 (Pin_31), J25.32 (Pin_32), J25.4 (Pin_4), J25.5 (Pin_5), J25.6 (Pin_6), J25.7 (Pin_7), J25.8 (Pin_8), J25.9 (Pin_9), J26.1 (Pin_1), J26.10 (Pin_10), J26.11 (Pin_11), J26.12 (Pin_12), J26.13 (Pin_13), J26.14 (Pin_14), J26.15 (Pin_15), J26.16 (Pin_16), J26.17 (Pin_17), J26.18 (Pin_18), J26.19 (Pin_19), J26.2 (Pin_2), J26.20 (Pin_20), J26.21 (Pin_21), J26.22 (Pin_22), J26.23 (Pin_23), J26.24 (Pin_24), J26.25 (Pin_25), J26.26 (Pin_26), J26.27 (Pin_27), J26.28 (Pin_28), J26.29 (Pin_29), J26.3 (Pin_3), J26.30 (Pin_30), J26.31 (Pin_31), J26.32 (Pin_32), J26.4 (Pin_4), J26.5 (Pin_5), J26.6 (Pin_6), J26.7 (Pin_7), J26.8 (Pin_8), J26.9 (Pin_9), J27.A10 (+3.3V), J27.A9 (+3.3V), J27.B10 (3.3Vaux), J27.B8 (+3.3V), R277.1, R279.1, R281.1, R283.1, R285.1, R287.1, R289.1, R291.1, R293.1, R295.1, R297.1, R299.1, R301.1, R303.1, R305.1, R307.1, R309.1, R311.1, R313.1, R315.1, R317.1, R319.1, R321.1, R323.1, R325.1, R327.1, R329.1, R331.1, R333.1, R335.1, R337.1, R339.1, R341.1, R343.1, R345.1, R347.1, R349.1, R351.1, R353.1, R355.1, R357.1, R359.1, R361.1, R363.1, R365.1, R367.1, R369.1, R371.1, R373.1, R375.1, R377.1, R379.1, R381.1, R383.1, R385.1, R387.1, R389.1, R391.1, R393.1, R395.1, R397.1, R399.1, R401.1, R403.1, R405.1, R407.1, R409.1, R411.1, R413.1
- new net CLK_PH0: J20.A13 (REFCLK+), J27.A13 (REFCLK+)
- new net CLK_PH1: J20.A14 (REFCLK-), J27.A14 (REFCLK-)
- new net GND: J18.10 (Pin_10), J18.2 (Pin_2), J18.4 (Pin_4), J18.6 (Pin_6), J18.8 (Pin_8), J19.10 (Pin_10), J19.12 (Pin_12), J19.14 (Pin_14), J19.16 (Pin_16), J19.18 (Pin_18), J19.2 (Pin_2), J19.20 (Pin_20), J19.22 (Pin_22), J19.24 (Pin_24), J19.26 (Pin_26), J19.28 (Pin_28), J19.30 (Pin_30), J19.32 (Pin_32), J19.34 (Pin_34), J19.36 (Pin_36), J19.38 (Pin_38), J19.4 (Pin_4), J19.40 (Pin_40), J19.42 (Pin_42), J19.44 (Pin_44), J19.46 (Pin_46), J19.48 (Pin_48), J19.50 (Pin_50), J19.52 (Pin_52), J19.54 (Pin_54), J19.56 (Pin_56), J19.58 (Pin_58), J19.6 (Pin_6), J19.60 (Pin_60), J19.62 (Pin_62), J19.64 (Pin_64), J19.8 (Pin_8), J20.A12 (GND), J20.A15 (GND), J20.A18 (GND), J20.A20 (GND), J20.A23 (GND), J20.A24 (GND), J20.A27 (GND), J20.A28 (GND), J20.A31 (GND), J20.A34 (GND), J20.A37 (GND), J20.A38 (GND), J20.A4 (GND), J20.A41 (GND), J20.A42 (GND), J20.A45 (GND), J20.A46 (GND), J20.A49 (GND), J20.A51 (GND), J20.A54 (GND), J20.A55 (GND), J20.A58 (GND), J20.A59 (GND), J20.A62 (GND), J20.A63 (GND), J20.A66 (GND), J20.A67 (GND), J20.A70 (GND), J20.A71 (GND), J20.A74 (GND), J20.A75 (GND), J20.A78 (GND), J20.A79 (GND), J20.A82 (GND), J20.B13 (GND), J20.B16 (GND), J20.B18 (GND), J20.B21 (GND), J20.B22 (GND), J20.B25 (GND), J20.B26 (GND), J20.B29 (GND), J20.B32 (GND), J20.B35 (GND), J20.B36 (GND), J20.B39 (GND), J20.B4 (GND), J20.B40 (GND), J20.B43 (GND), J20.B44 (GND), J20.B47 (GND), J20.B49 (GND), J20.B52 (GND), J20.B53 (GND), J20.B56 (GND), J20.B57 (GND), J20.B60 (GND), J20.B61 (GND), J20.B64 (GND), J20.B65 (GND), J20.B68 (GND), J20.B69 (GND), J20.B7 (GND), J20.B72 (GND), J20.B73 (GND), J20.B76 (GND), J20.B77 (GND), J20.B80 (GND), J21.10 (Pin_10), J21.2 (Pin_2), J21.4 (Pin_4), J21.6 (Pin_6), J21.8 (Pin_8), J22.10 (Pin_10), J22.2 (Pin_2), J22.4 (Pin_4), J22.6 (Pin_6), J22.8 (Pin_8), J23.10 (Pin_10), J23.12 (Pin_12), J23.14 (Pin_14), J23.16 (Pin_16), J23.18 (Pin_18), J23.2 (Pin_2), J23.20 (Pin_20), J23.22 (Pin_22), J23.24 (Pin_24), J23.26 (Pin_26), J23.28 (Pin_28), J23.30 (Pin_30), J23.32 (Pin_32), J23.34 (Pin_34), J23.36 (Pin_36), J23.38 (Pin_38), J23.4 (Pin_4), J23.40 (Pin_40), J23.42 (Pin_42), J23.44 (Pin_44), J23.46 (Pin_46), J23.48 (Pin_48), J23.50 (Pin_50), J23.52 (Pin_52), J23.54 (Pin_54), J23.56 (Pin_56), J23.58 (Pin_58), J23.6 (Pin_6), J23.60 (Pin_60), J23.62 (Pin_62), J23.64 (Pin_64), J23.8 (Pin_8), J27.A12 (GND), J27.A15 (GND), J27.A18 (GND), J27.A20 (GND), J27.A23 (GND), J27.A24 (GND), J27.A27 (GND), J27.A28 (GND), J27.A31 (GND), J27.A34 (GND), J27.A37 (GND), J27.A38 (GND), J27.A4 (GND), J27.A41 (GND), J27.A42 (GND), J27.A45 (GND), J27.A46 (GND), J27.A49 (GND), J27.A51 (GND), J27.A54 (GND), J27.A55 (GND), J27.A58 (GND), J27.A59 (GND), J27.A62 (GND), J27.A63 (GND), J27.A66 (GND), J27.A67 (GND), J27.A70 (GND), J27.A71 (GND), J27.A74 (GND), J27.A75 (GND), J27.A78 (GND), J27.A79 (GND), J27.A82 (GND), J27.B13 (GND), J27.B16 (GND), J27.B18 (GND), J27.B21 (GND), J27.B22 (GND), J27.B25 (GND), J27.B26 (GND), J27.B29 (GND), J27.B32 (GND), J27.B35 (GND), J27.B36 (GND), J27.B39 (GND), J27.B4 (GND), J27.B40 (GND), J27.B43 (GND), J27.B44 (GND), J27.B47 (GND), J27.B49 (GND), J27.B52 (GND), J27.B53 (GND), J27.B56 (GND), J27.B57 (GND), J27.B60 (GND), J27.B61 (GND), J27.B64 (GND), J27.B65 (GND), J27.B68 (GND), J27.B69 (GND), J27.B7 (GND), J27.B72 (GND), J27.B73 (GND), J27.B76 (GND), J27.B77 (GND), J27.B80 (GND), J3.10 (Pin_10), J3.2 (Pin_2), J3.4 (Pin_4), J3.6 (Pin_6), J3.8 (Pin_8), R278.2, R280.2, R282.2, R284.2, R286.2, R288.2, R290.2, R292.2, R294.2, R296.2, R298.2, R300.2, R302.2, R304.2, R306.2, R308.2, R310.2, R312.2, R314.2, R316.2, R318.2, R320.2, R322.2, R324.2, R326.2, R328.2, R330.2, R332.2, R334.2, R336.2, R338.2, R340.2, R342.2, R344.2, R346.2, R348.2, R350.2, R352.2, R354.2, R356.2, R358.2, R360.2, R362.2, R364.2, R366.2, R368.2, R370.2, R372.2, R374.2, R376.2, R378.2, R380.2, R382.2, R384.2, R386.2, R388.2, R390.2, R392.2, R394.2, R396.2, R398.2, R400.2, R402.2, R404.2, R406.2, R408.2, R410.2, R412.2, R414.2
- new net rsvda0: J20.B82 (RSVD), J21.1 (Pin_1), J27.B82 (RSVD)
- new net rsvda1: J20.A50 (RSVD), J21.3 (Pin_3), J27.A50 (RSVD)
- new net rsvda2: J20.A33 (RSVD), J21.5 (Pin_5), J27.A33 (RSVD)
- new net rsvda3: J20.B30 (RSVD), J21.7 (Pin_7), J27.B30 (RSVD)
- new net rsvda4: J20.A32 (RSVD), J21.9 (Pin_9), J27.A32 (RSVD)
- new net rsvda5: J20.A19 (RSVD), J27.A19 (RSVD), J3.1 (Pin_1)
- new net rsvda6: J20.B12 (RSVD), J27.B12 (RSVD), J3.3 (Pin_3)
- new net smclka: J20.B5 (SMCLK), J27.B5 (SMCLK), J3.7 (Pin_7)
- new net smdata: J20.B6 (SMDAT), J27.B6 (SMDAT), J3.9 (Pin_9)
- new net write0: D287.1 (K), D288.2 (A), J19.1 (Pin_1), J20.B14 (PETp0), J27.B14 (PETp0)
- new net write1: D295.1 (K), D296.2 (A), J19.3 (Pin_3), J20.B15 (PETn0), J27.B15 (PETn0)
- new net write10: D367.1 (K), D368.2 (A), J19.21 (Pin_21), J20.B37 (PETp5), J27.B37 (PETp5)
- new net write11: D375.1 (K), D376.2 (A), J19.23 (Pin_23), J20.B38 (PETn5), J27.B38 (PETn5)
- new net write12: D383.1 (K), D384.2 (A), J19.25 (Pin_25), J20.B41 (PETp6), J27.B41 (PETp6)
- new net write13: D391.1 (K), D392.2 (A), J19.27 (Pin_27), J20.B42 (PETn6), J27.B42 (PETn6)
- new net write14: D399.1 (K), D400.2 (A), J19.29 (Pin_29), J20.B45 (PETp7), J27.B45 (PETp7)
- new net write15: D407.1 (K), D408.2 (A), J19.31 (Pin_31), J20.B46 (PETn7), J27.B46 (PETn7)
- new net write16: D289.1 (K), D290.2 (A), J19.33 (Pin_33), J20.B50 (PETp8), J27.B50 (PETp8)
- new net write17: D297.1 (K), D298.2 (A), J19.35 (Pin_35), J20.B51 (PETn8), J27.B51 (PETn8)
- new net write18: D305.1 (K), D306.2 (A), J19.37 (Pin_37), J20.B54 (PETp9), J27.B54 (PETp9)
- new net write19: D313.1 (K), D314.2 (A), J19.39 (Pin_39), J20.B55 (PETn9), J27.B55 (PETn9)
- new net write2: D303.1 (K), D304.2 (A), J19.5 (Pin_5), J20.B19 (PETp1), J27.B19 (PETp1)
- new net write20: D321.1 (K), D322.2 (A), J19.41 (Pin_41), J20.B58 (PETp10), J27.B58 (PETp10)
- new net write21: D329.1 (K), D330.2 (A), J19.43 (Pin_43), J20.B59 (PETn10), J27.B59 (PETn10)
- new net write22: D337.1 (K), D338.2 (A), J19.45 (Pin_45), J20.B62 (PETp11), J27.B62 (PETp11)
- new net write23: D345.1 (K), D346.2 (A), J19.47 (Pin_47), J20.B63 (PETn11), J27.B63 (PETn11)
- new net write24: D353.1 (K), D354.2 (A), J19.49 (Pin_49), J20.B66 (PETp12), J27.B66 (PETp12)
- new net write25: D361.1 (K), D362.2 (A), J19.51 (Pin_51), J20.B67 (PETn12), J27.B67 (PETn12)
- new net write26: D369.1 (K), D370.2 (A), J19.53 (Pin_53), J20.B70 (PETp13), J27.B70 (PETp13)
- new net write27: D377.1 (K), D378.2 (A), J19.55 (Pin_55), J20.B71 (PETn13), J27.B71 (PETn13)
- new net write28: D385.1 (K), D386.2 (A), J19.57 (Pin_57), J20.B74 (PETp14), J27.B74 (PETp14)
- new net write29: D393.1 (K), D394.2 (A), J19.59 (Pin_59), J20.B75 (PETn14), J27.B75 (PETn14)
- new net write3: D311.1 (K), D312.2 (A), J19.7 (Pin_7), J20.B20 (PETn1), J27.B20 (PETn1)
- new net write30: D401.1 (K), D402.2 (A), J19.61 (Pin_61), J20.B78 (PETp15), J27.B78 (PETp15)
- new net write31: D409.1 (K), D410.2 (A), J19.63 (Pin_63), J20.B79 (PETn15), J27.B79 (PETn15)
- new net write32: D291.1 (K), D292.2 (A), J20.A16 (PERp0), J23.1 (Pin_1), J27.A16 (PERp0)
- new net write33: D299.1 (K), D300.2 (A), J20.A17 (PERn0), J23.3 (Pin_3), J27.A17 (PERn0)
- new net write34: D307.1 (K), D308.2 (A), J20.A21 (PERp1), J23.5 (Pin_5), J27.A21 (PERp1)
- new net write35: D315.1 (K), D316.2 (A), J20.A22 (PERn1), J23.7 (Pin_7), J27.A22 (PERn1)
- new net write36: D323.1 (K), D324.2 (A), J20.A25 (PERp2), J23.9 (Pin_9), J27.A25 (PERp2)
- new net write37: D331.1 (K), D332.2 (A), J20.A26 (PERn2), J23.11 (Pin_11), J27.A26 (PERn2)
- new net write38: D339.1 (K), D340.2 (A), J20.A29 (PERp3), J23.13 (Pin_13), J27.A29 (PERp3)
- new net write39: D347.1 (K), D348.2 (A), J20.A30 (PERn3), J23.15 (Pin_15), J27.A30 (PERn3)
- new net write4: D319.1 (K), D320.2 (A), J19.9 (Pin_9), J20.B23 (PETp2), J27.B23 (PETp2)
- new net write40: D355.1 (K), D356.2 (A), J20.A35 (PERp4), J23.17 (Pin_17), J27.A35 (PERp4)
- new net write41: D363.1 (K), D364.2 (A), J20.A36 (PERn4), J23.19 (Pin_19), J27.A36 (PERn4)
- new net write42: D371.1 (K), D372.2 (A), J20.A39 (PERp5), J23.21 (Pin_21), J27.A39 (PERp5)
- new net write43: D379.1 (K), D380.2 (A), J20.A40 (PERn5), J23.23 (Pin_23), J27.A40 (PERn5)
- new net write44: D387.1 (K), D388.2 (A), J20.A43 (PERp6), J23.25 (Pin_25), J27.A43 (PERp6)
- new net write45: D395.1 (K), D396.2 (A), J20.A44 (PERn6), J23.27 (Pin_27), J27.A44 (PERn6)
- new net write46: D403.1 (K), D404.2 (A), J20.A47 (PERp7), J23.29 (Pin_29), J27.A47 (PERp7)
- new net write47: D411.1 (K), D412.2 (A), J20.A48 (PERn7), J23.31 (Pin_31), J27.A48 (PERn7)
- new net write48: D293.1 (K), D294.2 (A), J20.A52 (PERp8), J23.33 (Pin_33), J27.A52 (PERp8)
- new net write49: D301.1 (K), D302.2 (A), J20.A53 (PERn8), J23.35 (Pin_35), J27.A53 (PERn8)
- new net write5: D327.1 (K), D328.2 (A), J19.11 (Pin_11), J20.B24 (PETn2), J27.B24 (PETn2)
- new net write50: D309.1 (K), D310.2 (A), J20.A56 (PERp9), J23.37 (Pin_37), J27.A56 (PERp9)
- new net write51: D317.1 (K), D318.2 (A), J20.A57 (PERn9), J23.39 (Pin_39), J27.A57 (PERn9)
- new net write52: D325.1 (K), D326.2 (A), J20.A60 (PERp10), J23.41 (Pin_41), J27.A60 (PERp10)
- new net write53: D333.1 (K), D334.2 (A), J20.A61 (PERn10), J23.43 (Pin_43), J27.A61 (PERn10)
- new net write54: D341.1 (K), D342.2 (A), J20.A64 (PERp11), J23.45 (Pin_45), J27.A64 (PERp11)
- new net write55: D349.1 (K), D350.2 (A), J20.A65 (PERn11), J23.47 (Pin_47), J27.A65 (PERn11)
- new net write56: D357.1 (K), D358.2 (A), J20.A68 (PERp12), J23.49 (Pin_49), J27.A68 (PERp12)
- new net write57: D365.1 (K), D366.2 (A), J20.A69 (PERn12), J23.51 (Pin_51), J27.A69 (PERn12)
- new net write58: D373.1 (K), D374.2 (A), J20.A72 (PERp13), J23.53 (Pin_53), J27.A72 (PERp13)
- new net write59: D381.1 (K), D382.2 (A), J20.A73 (PERn13), J23.55 (Pin_55), J27.A73 (PERn13)
- new net write6: D335.1 (K), D336.2 (A), J19.13 (Pin_13), J20.B27 (PETp3), J27.B27 (PETp3)
- new net write60: D389.1 (K), D390.2 (A), J20.A76 (PERp14), J23.57 (Pin_57), J27.A76 (PERp14)
- new net write61: D397.1 (K), D398.2 (A), J20.A77 (PERn14), J23.59 (Pin_59), J27.A77 (PERn14)
- new net write62: D405.1 (K), D406.2 (A), J20.A80 (PERp15), J23.61 (Pin_61), J27.A80 (PERp15)
- new net write63: D413.1 (K), D414.2 (A), J20.A81 (PERn15), J23.63 (Pin_63), J27.A81 (PERn15)
- new net write7: D343.1 (K), D344.2 (A), J19.15 (Pin_15), J20.B28 (PETn3), J27.B28 (PETn3)
- new net write8: D351.1 (K), D352.2 (A), J19.17 (Pin_17), J20.B33 (PETp4), J27.B33 (PETp4)
- new net write9: D359.1 (K), D360.2 (A), J19.19 (Pin_19), J20.B34 (PETn4), J27.B34 (PETn4)
- new net writesel0: D277.1 (K), D278.2 (A), J20.B9 (JTAG1), J22.1 (Pin_1), J27.B9 (JTAG1)
- new net writesel1: D279.1 (K), D280.2 (A), J20.A5 (JTAG2), J22.3 (Pin_3), J27.A5 (JTAG2)
- new net writesel2: D281.1 (K), D282.2 (A), J20.A6 (JTAG3), J22.5 (Pin_5), J27.A6 (JTAG3)
- new net writesel3: D283.1 (K), D284.2 (A), J20.A7 (JTAG4), J22.7 (Pin_7), J27.A7 (JTAG4)
- new net writesel4: D285.1 (K), D286.2 (A), J20.A8 (JTAG5), J22.9 (Pin_9), J27.A8 (JTAG5)
- new net ~{RDT}: J20.A11 (~{PERST}), J27.A11 (~{PERST})
- new net ~{prsnt1}: J18.1 (Pin_1), J20.A1 (~{PRSNT1}), J27.A1 (~{PRSNT1})
- new net ~{prsnt2}: J18.3 (Pin_3), J20.B17 (~{PRSNT2}), J27.B17 (~{PRSNT2})
- new net ~{prsnt3}: J18.5 (Pin_5), J20.B31 (~{PRSNT2}), J27.B31 (~{PRSNT2})
- new net ~{prsnt4}: J18.7 (Pin_7), J20.B48 (~{PRSNT2}), J27.B48 (~{PRSNT2})
- new net ~{prsnt5}: J18.9 (Pin_9), J20.B81 (~{PRSNT2}), J27.B81 (~{PRSNT2})
- new net ~{wakea}: J20.B11 (~{WAKE}), J27.B11 (~{WAKE}), J3.5 (Pin_5)
Other:
- note added: "HI IND"
- note added: "LO IND"
